File: Thermo_CTRL_Unit.kicad_pcb (KiCad board)
At the start: 2 copper layers, 50 x 50 mm, 51 parts, among them IC1 ATMEGA168PA-A, J1 RJ12, P1 SW_TH1, P10 SW_TH6, P11 SW_W1, P12 SW_W2, P13 SW_W3, P14 SW_W4, P15 CONN_01X05, P2 ISCP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

Commit message: PCB Update
Parts:
- removed P10: SW_TH6, BK_Common:JST_B3B-XH-A
- removed P8: SW_TH5, BK_Common:JST_B3B-XH-A
- moved C5 104.6 mm to (113.5, 85.1), turned to 180 degrees
- moved D3 104.1 mm to (100.1, 110.3), turned to 90 degrees
- moved D1 103.8 mm to (104.2, 110.3), turned to 90 degrees
- moved D2 102.3 mm to (102.1, 110.3), turned to 90 degrees
- moved R15 96.0 mm to (121.2, 85.3)
- moved D4 95.7 mm to (106.2, 110.3), turned to 90 degrees
- moved R7 94.3 mm to (98.0, 106.7), turned to 270 degrees
- moved P11 93.8 mm to (94.0, 99.6), turned to 270 degrees
- moved R6 88.3 mm to (98.0, 103.4), turned to 90 degrees
- moved R5 86.2 mm to (123.6, 81.5)
- moved R9 85.3 mm to (112.8, 111.5)
- moved R4 85.0 mm to (128.2, 82.3)
- moved P12 83.0 mm to (94.0, 108.2), turned to 270 degrees
- moved R8 80.5 mm to (109.2, 111.5), turned to 180 degrees
- moved P13 69.4 mm to (110.0, 116.1)
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Connections:
- IC1 pad 19: /TH_5 -> /TH_3
- IC1 pad 22: /TH_6 -> /TH_4
- IC1 pad 25: /TH_3 -> /SW_SH1
- IC1 pad 26: /TH_4 -> /SW_SH2
- IC1 pad 27: /SW_SH1 -> (no net)
- IC1 pad 28: /SW_SH2 -> (no net)
- R11 pad 2: Net-(R11-Pad2) -> GND
- R12 pad 2: Net-(R11-Pad2) -> GND
- R13 pad 2: Net-(R11-Pad2) -> GND
- R14 pad 2: Net-(R11-Pad2) -> GND

Commit message: SCH change
Parts:
- added C10: 10uF, Capacitors_SMD:C_1206, F.Cu at (92.8, 94.0)
- added C11: 100nF, Capacitors_SMD:C_0805, F.Cu at (103.1, 86.1)
- added C12: 1uF, Capacitors_SMD:C_1206, F.Cu at (103.1, 90.4)
- added C13: 10uF, Capacitors_SMD:C_1206, F.Cu at (125.1, 89.5)
- added D6: SS13, Diodes_SMD:SMA_Standard, F.Cu at (99.1, 99.0)
- added P10: IIC, Pin_Headers:Pin_Header_Straight_1x04, F.Cu at (128.4, 100.6)
- added P8: VIN, Pin_Headers:Pin_Header_Straight_1x02, F.Cu at (92.3, 89.6)
- added R17: 1K, Resistors_SMD:R_0805, F.Cu at (131.5, 96.0)
- added R18: 1K, Resistors_SMD:R_0805, F.Cu at (131.5, 106.7)
- added REF**: Symbol_OSHW-Logo_SilkScreen, Symbols:Symbol_OSHW-Logo_SilkScreen, F.Cu at (128.0, 109.2)
- added REF**: Symbol_OSHW-Logo_CopperTop, BK_Common:Symbol_OSHW-Logo_CopperTop_MASK, B.Cu at (128.0, 109.2)
- added U2: MC78M05CDT, TO_SOT_Packages_SMD:TO-252-2Lead, F.Cu at (98.2, 93.6)
- added U3: HT7333-A, TO_SOT_Packages_SMD:SOT89-3_Housing, F.Cu at (125.1, 85.2)
- moved R4 9.70 mm to (119.3, 86.0)
- moved P2 5.23 mm to (131.1, 115.4), turned to 270 degrees
- moved R5 5.00 mm to (119.3, 83.9)
- moved C5 3.44 mm to (112.0, 88.1)
- moved R15 3.38 mm to (119.3, 88.1)
- moved P4 2.88 mm to (106.2, 82.5)
- moved SW1 2.70 mm to (115.5, 91.3)
- moved C1 1.11 mm to (107.1, 102.6)
- moved C2 1.11 mm to (107.1, 98.5)
- moved C3 1.11 mm to (103.6, 97.7)
- moved C4 1.11 mm to (103.6, 103.8)
- moved X1 1.11 mm to (103.6, 100.8)
- moved R6 0.88 mm to (98.9, 103.7), turned to 0 degrees
Connections:
- IC1 pad 27: (no net) -> /SDA
- IC1 pad 28: (no net) -> /SCL
- J1 pad 1: (no net) -> Net-(J1-Pad1)
- J1 pad 6: (no net) -> Net-(J1-Pad6)
Routing:
- net +5V: track 0.00 -> 289.7 mm, vias 0 -> 7
- net GND: track 0.00 -> 103.9 mm, vias 0 -> 7
- net /RST: track 0.00 -> 63.3 mm, vias 0 -> 5
- net /ZCD: track 0.00 -> 36.5 mm, vias 0 -> 2
- net /RxD: track 0.00 -> 29.9 mm
- net /TH_2: track 0.00 -> 29.1 mm
- net /SW_SH1: track 0.00 -> 27.0 mm
- net /TxD: track 0.00 -> 25.9 mm, vias 0 -> 2
- net /SW_W1: track 0.00 -> 24.6 mm
- net /TH_4: track 0.00 -> 23.3 mm
- net /SW_SH2: track 0.00 -> 23.2 mm
- net /MISO: track 0.00 -> 22.8 mm
- net /Triac_3: track 0.00 -> 22.7 mm
- net /MOSI: track 0.00 -> 22.7 mm
- net /TH_3: track 0.00 -> 21.5 mm
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- added copper zone on B.Cu, net GND
Other:
- net class power added: clearance 0.2, trace_width 0.4, via_dia 0.6, via_drill 0.4
- rule pad_to_mask_clearance: 0.2 -> 0
- board text added: "BK 2016"
- board text added: "SENS NODE V1"

Commit message: PCB Change
Parts:
- C1: value 100n -> 1u
- moved C5 11.2 mm to (122.7, 91.3), turned to 90 degrees
- moved C13 2.90 mm to (127.4, 87.7)
- moved U3 2.90 mm to (127.4, 83.4)
Connections:
- J1 pad 1: Net-(J1-Pad1) -> (no net)
- J1 pad 6: Net-(J1-Pad6) -> (no net)
Routing:
- net +5V: track 289.7 -> 265.4 mm
- net /RST: track 63.3 -> 58.2 mm, vias 5 -> 3
- net GND: track 103.9 -> 107.8 mm
- net +3V3: track 15.8 -> 19.0 mm
- net /TH_2: track 29.1 -> 31.1 mm
- net /TxD: track 25.9 -> 25.1 mm
- net /SW_W2: track 21.1 -> 21.8 mm, vias 0 -> 1
- net /SW_W1: track 24.6 -> 24.7 mm, vias 0 -> 1
Other:
- board text added: "J1 RS-485: 2 - GND 3 - A 4 - B 5 - 5V"
- board text added: "P1,P3,P5,P7: Analog 1 - 5V 2 - An_In 3 - GND"
- board text added: "P10 IIC: 1 - 3.3V 2 - GND 3 - SCL 4 - SDA"
- board text added: "P11,P12,P13,14: Digital In (5v) Pullup 1 - Dig In 2 - GND"
- board text added: "P15 TTL SER: 1 - 5V 2 - RxD 3 - TXD 4 - DTR(rst) 5 - GND"
- board text added: "P6 ZCD Triac: 1 - 5V 2 - GND 3 - ZCD 4,5,6 - Triac"
- board text added: "P9 SW Input: Pullup 1 - SW1 2 - SW2 3 - GND"
